File: ifm-spark-dev.sch (KiCad schematic (older format))
At the start: 21 parts

Commit message: Annotated schematic
Parts:
- gave numbers to parts that had none: 21
Changed lines of the file:
@@
 $EndDescr
 $Comp
-L STM32F030x4 U?
+L STM32F030x4 U1
 U 1 1 59251F3D
 P 5550 3500
-F 0 "U?" H 6000 2400 60  0000 C CNN
+F 0 "U1" H 6000 2400 60  0000 C CNN
 F 1 "STM32F030x4" H 5500 3850 60  0000 C CNN
 F 2 "" H 5550 3700 60  0001 C CNN
@@
 $EndComp
 $Comp
-L +3.3V #PWR?
+L +3.3V #PWR7
 U 1 1 59251F94
 P 5500 1250
-F 0 "#PWR?" H 5500 1100 50  0001 C CNN
+F 0 "#PWR7" H 5500 1100 50  0001 C CNN
 F 1 "+3.3V" H 5500 1390 50  0000 C CNN
 F 2 "" H 5500 1250 50  0001 C CNN
@@
 $EndComp
 $Comp
-L GND #PWR?
+L GND #PWR8
 U 1 1 59251FDD
 P 5550 4950
-F 0 "#PWR?" H 5550 4700 50  0001 C CNN
+F 0 "#PWR8" H 5550 4700 50  0001 C CNN
 F 1 "GND" H 5550 4800 50  0000 C CNN
 F 2 "" H 5550 4950 50  0001 C CNN
@@
 $EndComp
 $Comp
-L C C?
+L C C2
 U 1 1 59252063
 P 3850 3350
-F 0 "C?" H 3875 3450 50  0000 L CNN
+F 0 "C2" H 3875 3450 50  0000 L CNN
 F 1 "20pF" H 3875 3250 50  0000 L CNN
 F 2 "" H 3888 3200 50  0001 C CNN
@@
 $EndComp
 $Comp
-L C C?
+L C C3
 U 1 1 592520BE
 P 3850 3650
-F 0 "C?" H 3875 3750 50  0000 L CNN
+F 0 "C3" H 3875 3750 50  0000 L CNN
 F 1 "20pF" H 3875 3550 50  0000 L CNN
 F 2 "" H 3888 3500 50  0001 C CNN
@@
 $EndComp
 $Comp
-L GND #PWR?
+L GND #PWR5
 U 1 1 5925217D
 P 3600 3750
-F 0 "#PWR?" H 3600 3500 50  0001 C CNN
+F 0 "#PWR5" H 3600 3500 50  0001 C CNN
 F 1 "GND" H 3600 3600 50  0000 C CNN
 F 2 "" H 3600 3750 50  0001 C CNN
@@
 Connection ~ 3600 3650
 $Comp
-L Crystal Y?
+L Crystal Y1
 U 1 1 592521E6
 P 4200 3500
-F 0 "Y?" H 4200 3650 50  0000 C CNN
+F 0 "Y1" H 4200 3650 50  0000 C CNN
 F 1 "8MHz" H 4200 3350 50  0000 C CNN
 F 2 "" H 4200 3500 50  0001 C CNN
@@
 	6250 4350 6400 4350
 $Comp
-L CONN_01X03_MALE J?
+L CONN_01X03_MALE J5
 U 1 1 59299BA5
 P 10350 1650
-F 0 "J?" H 10350 1925 50  0000 C CNN
+F 0 "J5" H 10350 1925 50  0000 C CNN
 F 1 "CONN_01X03_MALE" H 10375 1375 50  0000 C CNN
 F 2 "" H 10350 1850 50  0001 C CNN
@@
 	10050 1650 9900 1650
 $Comp
-L +3.3V #PWR?
+L +3.3V #PWR14
 U 1 1 59299D01
 P 9900 1200
-F 0 "#PWR?" H 9900 1050 50  0001 C CNN
+F 0 "#PWR14" H 9900 1050 50  0001 C CNN
 F 1 "+3.3V" H 9900 1340 50  0000 C CNN
 F 2 "" H 9900 1200 50  0001 C CNN
@@
 $EndComp
 $Comp
-L GND #PWR?
+L GND #PWR15
 U 1 1 59299D1B
 P 9900 2000
-F 0 "#PWR?" H 9900 1750 50  0001 C CNN
+F 0 "#PWR15" H 9900 1750 50  0001 C CNN
 F 1 "GND" H 9900 1850 50  0000 C CNN
 F 2 "" H 9900 2000 50  0001 C CNN
@@
 	11100 650  9300 650
 $Comp
-L C C?
+L C C5
 U 1 1 5929A23D
 P 6250 1700
-F 0 "C?" H 6275 1800 50  0000 L CNN
+F 0 "C5" H 6275 1800 50  0000 L CNN
 F 1 "10nF" H 6275 1600 50  0000 L CNN
 F 2 "" H 6288 1550 50  0001 C CNN
@@
 	5850 1450 5850 1550
 $Comp
-L GND #PWR?
+L GND #PWR10
 U 1 1 5929A301
 P 5850 2100
-F 0 "#PWR?" H 5850 1850 50  0001 C CNN
+F 0 "#PWR10" H 5850 1850 50  0001 C CNN
 F 1 "GND" H 5850 1950 50  0000 C CNN
 F 2 "" H 5850 2100 50  0001 C CNN
@@
 	5850 1950 5850 2100
 $Comp
-L CP C?
+L CP C4
 U 1 1 5929A34D
 P 5850 1700
-F 0 "C?" H 5875 1800 50  0000 L CNN
+F 0 "C4" H 5875 1800 50  0000 L CNN
 F 1 "1uF" H 5875 1600 50  0000 L CNN
 F 2 "" H 5888 1550 50  0001 C CNN
@@
 Connection ~ 5850 1950
 $Comp
-L +3.3V #PWR?
+L +3.3V #PWR9
 U 1 1 5929A588
 P 5850 1250
-F 0 "#PWR?" H 5850 1100 50  0001 C CNN
+F 0 "#PWR9" H 5850 1100 50  0001 C CNN
 F 1 "+3.3V" H 5850 1390 50  0000 C CNN
 F 2 "" H 5850 1250 50  0001 C CNN
@@
 $EndComp
 $Comp
-L R R?
+L R R3
 U 1 1 5929A77F
 P 4550 3650
-F 0 "R?" V 4630 3650 50  0000 C CNN
+F 0 "R3" V 4630 3650 50  0000 C CNN
 F 1 "390" V 4550 3650 50  0000 C CNN
 F 2 "" V 4480 3650 50  0001 C CNN
@@
 $EndComp
 $Comp
-L PTS525-SM15 SW?
+L PTS525-SM15 SW1
 U 1 1 592A4BF6
 P 3400 4200
-F 0 "SW?" H 3400 4400 60  0000 C CNN
+F 0 "SW1" H 3400 4400 60  0000 C CNN
 F 1 "PTS525-SM15" H 3400 4000 60  0000 C CNN
 F 2 "" H 3400 4200 60  0001 C CNN
@@
 	4400 4050 4850 4050
 $Comp
-L C C?
+L C C1
 U 1 1 592A4D64
 P 2750 4350
-F 0 "C?" H 2775 4450 50  0000 L CNN
+F 0 "C1" H 2775 4450 50  0000 L CNN
 F 1 "100nF" H 2775 4250 50  0000 L CNN
 F 2 "" H 2788 4200 50  0001 C CNN
@@
 $EndComp
 $Comp
-L GND #PWR?
+L GND #PWR4
 U 1 1 592A4E5A
 P 3400 4850
-F 0 "#PWR?" H 3400 4600 50  0001 C CNN
+F 0 "#PWR4" H 3400 4600 50  0001 C CNN
 F 1 "GND" H 3400 4700 50  0000 C CNN
 F 2 "" H 3400 4850 50  0001 C CNN
@@
 $EndComp
 $Comp
-L R R?
+L R R2
 U 1 1 592A4FC2
 P 4050 2900
-F 0 "R?" V 4130 2900 50  0000 C CNN
+F 0 "R2" V 4130 2900 50  0000 C CNN
 F 1 "10K" V 4050 2900 50  0000 C CNN
 F 2 "" V 3980 2900 50  0001 C CNN
@@
 	3800 4650 3800 4350
 $Comp
-L CONN_01X03_MALE J?
+L CONN_01X03_MALE J1
 U 1 1 592A5A04
 P 2950 2900
-F 0 "J?" H 2950 3175 50  0000 C CNN
+F 0 "J1" H 2950 3175 50  0000 C CNN
 F 1 "CONN_01X03_MALE" H 2975 2625 50  0000 C CNN
 F 2 "" H 2950 3100 50  0001 C CNN
@@
 $EndComp
 $Comp
-L +3.3V #PWR?
+L +3.3V #PWR2
 U 1 1 592A5ADB
 P 3400 2500
-F 0 "#PWR?" H 3400 2350 50  0001 C CNN
+F 0 "#PWR2" H 3400 2350 50  0001 C CNN
 F 1 "+3.3V" H 3400 2640 50  0000 C CNN
 F 2 "" H 3400 2500 50  0001 C CNN
@@
 $EndComp
 $Comp
-L GND #PWR?
+L GND #PWR3
 U 1 1 592A5B0A
 P 3400 3300
-F 0 "#PWR?" H 3400 3050 50  0001 C CNN
+F 0 "#PWR3" H 3400 3050 50  0001 C CNN
 F 1 "GND" H 3400 3150 50  0000 C CNN
 F 2 "" H 3400 3300 50  0001 C CNN
@@
 	5500 1800 5500 2200
 $Comp
-L CONN_01X07 J?
+L CONN_01X07 J4
 U 1 1 592A6D68
 P 8000 3650
-F 0 "J?" H 8000 4050 50  0000 C CNN
+F 0 "J4" H 8000 4050 50  0000 C CNN
 F 1 "CONN_01X07" V 8100 3650 50  0000 C CNN
 F 2 "" H 8000 3650 50  0001 C CNN
@@
 $EndComp
 $Comp
-L +3.3V #PWR?
+L +3.3V #PWR12
 U 1 1 592A6DD6
 P 7250 3200
-F 0 "#PWR?" H 7250 3050 50  0001 C CNN
+F 0 "#PWR12" H 7250 3050 50  0001 C CNN
 F 1 "+3.3V" H 7250 3340 50  0000 C CNN
 F 2 "" H 7250 3200 50  0001 C CNN
@@
 	7300 3900 6250 3900
 $Comp
-L GND #PWR?
+L GND #PWR11
 U 1 1 592A6F95
 P 7150 3600
-F 0 "#PWR?" H 7150 3350 50  0001 C CNN
+F 0 "#PWR11" H 7150 3350 50  0001 C CNN
 F 1 "GND" H 7150 3450 50  0000 C CNN
 F 2 "" H 7150 3600 50  0001 C CNN
@@
 	8250 3000 6250 3000
 $Comp
-L CONN_01X06 J?
+L CONN_01X06 J2
 U 1 1 592BABFC
 P 6650 3400
-F 0 "J?" H 6650 3750 50  0000 C CNN
+F 0 "J2" H 6650 3750 50  0000 C CNN
 F 1 "CONN_01X06" V 6750 3400 50  0000 C CNN
 F 2 "" H 6650 3400 50  0001 C CNN
@@
 	6250 3650 6450 3650
 $Comp
-L R R?
+L R R4
 U 1 1 594DDEF4
 P 5150 1800
-F 0 "R?" V 5230 1800 50  0000 C CNN
+F 0 "R4" V 5230 1800 50  0000 C CNN
 F 1 "1K" V 5150 1800 50  0000 C CNN
 F 2 "" V 5080 1800 50  0001 C CNN
@@
 $EndComp
 $Comp
-L LED D?
+L LED D1
 U 1 1 594DDF53
 P 4800 2050
-F 0 "D?" H 4800 2150 50  0000 C CNN
+F 0 "D1" H 4800 2150 50  0000 C CNN
 F 1 "LED" H 4800 1950 50  0000 C CNN
 F 2 "" H 4800 2050 50  0001 C CNN
@@
 $EndComp
 $Comp
-L GND #PWR?
+L GND #PWR6
 U 1 1 594DDFC0
 P 4800 2300
-F 0 "#PWR?" H 4800 2050 50  0001 C CNN
+F 0 "#PWR6" H 4800 2050 50  0001 C CNN
 F 1 "GND" H 4800 2150 50  0000 C CNN
 F 2 "" H 4800 2300 50  0001 C CNN
@@
 BOOT0
 $Comp
-L CONN_01X02 J?
+L CONN_01X02 J3
 U 1 1 594DF673
 P 6750 2650
-F 0 "J?" H 6750 2800 50  0000 C CNN
+F 0 "J3" H 6750 2800 50  0000 C CNN
 F 1 "CONN_01X02" V 6850 2650 50  0000 C CNN
 F 2 "" H 6750 2650 50  0001 C CNN
@@
 RX
 $Comp
-L R R?
+L R R5
 U 1 1 594E146B
 P 5600 1850
-F 0 "R?" V 5680 1850 50  0000 C CNN
+F 0 "R5" V 5680 1850 50  0000 C CNN
 F 1 "0" V 5600 1850 50  0000 C CNN
 F 2 "" V 5530 1850 50  0001 C CNN
@@
 	5600 2200 5600 2000
 $Comp
-L R R?
+L R R1
 U 1 1 594E20A6
 P 2750 3800
-F 0 "R?" V 2830 3800 50  0000 C CNN
+F 0 "R1" V 2830 3800 50  0000 C CNN
 F 1 "1K" V 2750 3800 50  0000 C CNN
 F 2 "" V 2680 3800 50  0001 C CNN
@@
 $EndComp
 $Comp
-L +3.3V #PWR?
+L +3.3V #PWR1
 U 1 1 594E214F
 P 2750 3600
-F 0 "#PWR?" H 2750 3450 50  0001 C CNN
+F 0 "#PWR1" H 2750 3450 50  0001 C CNN
 F 1 "+3.3V" H 2750 3740 50  0000 C CNN
 F 2 "" H 2750 3600 50  0001 C CNN
@@
 PA4
 $Comp
-L R R?
+L R R6
 U 1 1 594E286C
 P 8750 1250
-F 0 "R?" V 8830 1250 50  0000 C CNN
+F 0 "R6" V 8830 1250 50  0000 C CNN
 F 1 "1K" V 8750 1250 50  0000 C CNN
 F 2 "" V 8680 1250 50  0001 C CNN
@@
 $EndComp
 $Comp
-L LED D?
+L LED D2
 U 1 1 594E28B5
 P 8750 1650
-F 0 "D?" H 8750 1750 50  0000 C CNN
+F 0 "D2" H 8750 1750 50  0000 C CNN
 F 1 "LED" H 8750 1550 50  0000 C CNN
 F 2 "" H 8750 1650 50  0001 C CNN
@@
 $EndComp
 $Comp
-L GND #PWR?
+L GND #PWR13
 U 1 1 594E29ED
 P 8750 1950
-F 0 "#PWR?" H 8750 1700 50  0001 C CNN
+F 0 "#PWR13" H 8750 1700 50  0001 C CNN
 F 1 "GND" H 8750 1800 50  0000 C CNN
 F 2 "" H 8750 1950 50  0001 C CNN

Commit message: Associated all the easy passives and pin headers
Parts:
- C1, C2, C3, C4, C5: footprint (none) -> Capacitors_SMD:C_0805_HandSoldering
- D1, D2: footprint (none) -> LEDs:LED_0805
- J1, J5: footprint (none) -> Pin_Headers:Pin_Header_Straight_1x03_Pitch2.54mm
- J2: footprint (none) -> Pin_Headers:Pin_Header_Straight_1x06_Pitch2.54mm
- J3: footprint (none) -> Pin_Headers:Pin_Header_Straight_1x02_Pitch2.54mm
- J4: footprint (none) -> Pin_Headers:Pin_Header_Straight_1x07_Pitch2.54mm
- R1, R2, R3, R4, R5, R6: footprint (none) -> Resistors_SMD:R_0805_HandSoldering
Changed lines of the file:
@@
 $EndComp
 $Comp
-L +3.3V #PWR7
+L +3.3V #PWR01
 U 1 1 59251F94
 P 5500 1250
-F 0 "#PWR7" H 5500 1100 50  0001 C CNN
+F 0 "#PWR01" H 5500 1100 50  0001 C CNN
 F 1 "+3.3V" H 5500 1390 50  0000 C CNN
 F 2 "" H 5500 1250 50  0001 C CNN
@@
 $EndComp
 $Comp
-L GND #PWR8
+L GND #PWR02
 U 1 1 59251FDD
 P 5550 4950
-F 0 "#PWR8" H 5550 4700 50  0001 C CNN
+F 0 "#PWR02" H 5550 4700 50  0001 C CNN
 F 1 "GND" H 5550 4800 50  0000 C CNN
 F 2 "" H 5550 4950 50  0001 C CNN
@@
 F 0 "C2" H 3875 3450 50  0000 L CNN
 F 1 "20pF" H 3875 3250 50  0000 L CNN
-F 2 "" H 3888 3200 50  0001 C CNN
+F 2 "Capacitors_SMD:C_0805_HandSoldering" H 3888 3200 50  0001 C CNN
 F 3 "" H 3850 3350 50  0001 C CNN
 	1    3850 3350
@@
 F 0 "C3" H 3875 3750 50  0000 L CNN
 F 1 "20pF" H 3875 3550 50  0000 L CNN
-F 2 "" H 3888 3500 50  0001 C CNN
+F 2 "Capacitors_SMD:C_0805_HandSoldering" H 3888 3500 50  0001 C CNN
 F 3 "" H 3850 3650 50  0001 C CNN
 	1    3850 3650
@@
 $EndComp
 $Comp
-L GND #PWR5
+L GND #PWR03
 U 1 1 5925217D
 P 3600 3750
-F 0 "#PWR5" H 3600 3500 50  0001 C CNN
+F 0 "#PWR03" H 3600 3500 50  0001 C CNN
 F 1 "GND" H 3600 3600 50  0000 C CNN
 F 2 "" H 3600 3750 50  0001 C CNN
@@
 	3700 3350 3600 3350
 Wire Wire Line
-	3600 3350 3600 3650
-Wire Wire Line
-	3600 3650 3600 3750
+	3600 3350 3600 3750
 Wire Wire Line
 	3700 3650 3600 3650
@@
 F 0 "J5" H 10350 1925 50  0000 C CNN
 F 1 "CONN_01X03_MALE" H 10375 1375 50  0000 C CNN
-F 2 "" H 10350 1850 50  0001 C CNN
+F 2 "Pin_Headers:Pin_Header_Straight_1x03_Pitch2.54mm" H 10350 1850 50  0001 C CNN
 F 3 "" H 10350 1850 50  0001 C CNN
 	1    10350 1650
@@
 	10050 1650 9900 1650
 $Comp
-L +3.3V #PWR14
+L +3.3V #PWR04
 U 1 1 59299D01
 P 9900 1200
-F 0 "#PWR14" H 9900 1050 50  0001 C CNN
+F 0 "#PWR04" H 9900 1050 50  0001 C CNN
 F 1 "+3.3V" H 9900 1340 50  0000 C CNN
 F 2 "" H 9900 1200 50  0001 C CNN
@@
 $EndComp
 $Comp
-L GND #PWR15
+L GND #PWR05
 U 1 1 59299D1B
 P 9900 2000
-F 0 "#PWR15" H 9900 1750 50  0001 C CNN
+F 0 "#PWR05" H 9900 1750 50  0001 C CNN
 F 1 "GND" H 9900 1850 50  0000 C CNN
 F 2 "" H 9900 2000 50  0001 C CNN
@@
 F 0 "C5" H 6275 1800 50  0000 L CNN
 F 1 "10nF" H 6275 1600 50  0000 L CNN
-F 2 "" H 6288 1550 50  0001 C CNN
+F 2 "Capacitors_SMD:C_0805_HandSoldering" H 6288 1550 50  0001 C CNN
 F 3 "" H 6250 1700 50  0001 C CNN
 	1    6250 1700
@@
 $EndComp
 Wire Wire Line
-	5850 1250 5850 1450
-Wire Wire Line
-	5850 1450 5850 1550
-$Comp
-L GND #PWR10
+	5850 1250 5850 1550
+$Comp
+L GND #PWR06
 U 1 1 5929A301
 P 5850 2100
-F 0 "#PWR10" H 5850 1850 50  0001 C CNN
+F 0 "#PWR06" H 5850 1850 50  0001 C CNN
 F 1 "GND" H 5850 1950 50  0000 C CNN
 F 2 "" H 5850 2100 50  0001 C CNN
@@
 $EndComp
 Wire Wire Line
-	5850 1850 5850 1950
-Wire Wire Line
-	5850 1950 5850 2100
+	5850 1850 5850 2100
 $Comp
 L CP C4
@@
 F 0 "C4" H 5875 1800 50  0000 L CNN
 F 1 "1uF" H 5875 1600 50  0000 L CNN
-F 2 "" H 5888 1550 50  0001 C CNN
+F 2 "Capacitors_SMD:C_0805_HandSoldering" H 5888 1550 50  0001 C CNN
 F 3 "" H 5850 1700 50  0001 C CNN
 	1    5850 1700
@@
 $EndComp
 Wire Wire Line
-	5600 1450 5850 1450
-Wire Wire Line
-	5850 1450 6250 1450
+	5600 1450 6250 1450
 Wire Wire Line
 	6250 1450 6250 1550
@@
 Connection ~ 5850 1950
 $Comp
-L +3.3V #PWR9
+L +3.3V #PWR07
 U 1 1 5929A588
 P 5850 1250
-F 0 "#PWR9" H 5850 1100 50  0001 C CNN
+F 0 "#PWR07" H 5850 1100 50  0001 C CNN
 F 1 "+3.3V" H 5850 1390 50  0000 C CNN
 F 2 "" H 5850 1250 50  0001 C CNN
@@
 F 0 "R3" V 4630 3650 50  0000 C CNN
 F 1 "390" V 4550 3650 50  0000 C CNN
-F 2 "" V 4480 3650 50  0001 C CNN
+F 2 "Resistors_SMD:R_0805_HandSoldering" V 4480 3650 50  0001 C CNN
 F 3 "" H 4550 3650 50  0001 C CNN
 	1    4550 3650
@@
 $EndComp
 Wire Wire Line
-	3750 4050 4400 4050
-Wire Wire Line
-	4400 4050 4850 4050
+	3750 4050 4850 4050
 $Comp
 L C C1
@@
 F 0 "C1" H 2775 4450 50  0000 L CNN
 F 1 "100nF" H 2775 4250 50  0000 L CNN
-F 2 "" H 2788 4200 50  0001 C CNN
+F 2 "Capacitors_SMD:C_0805_HandSoldering" H 2788 4200 50  0001 C CNN
 F 3 "" H 2750 4350 50  0001 C CNN
 	1    2750 4350
@@
 $EndComp
 $Comp
-L GND #PWR4
+L GND #PWR08
 U 1 1 592A4E5A
 P 3400 4850
-F 0 "#PWR4" H 3400 4600 50  0001 C CNN
+F 0 "#PWR08" H 3400 4600 50  0001 C CNN
 F 1 "GND" H 3400 4700 50  0000 C CNN
 F 2 "" H 3400 4850 50  0001 C CNN
@@
 F 0 "R2" V 4130 2900 50  0000 C CNN
 F 1 "10K" V 4050 2900 50  0000 C CNN
-F 2 "" V 3980 2900 50  0001 C CNN
+F 2 "Resistors_SMD:R_0805_HandSoldering" V 3980 2900 50  0001 C CNN
 F 3 "" H 4050 2900 50  0001 C CNN
 	1    4050 2900
@@
 	3050 4050 2750 4050
 Wire Wire Line
-	2750 3950 2750 4050
-Wire Wire Line
-	2750 4050 2750 4200
+	2750 3950 2750 4200
 Wire Wire Line
 	3750 4350 3800 4350
@@
 F 0 "J1" H 2950 3175 50  0000 C CNN
 F 1 "CONN_01X03_MALE" H 2975 2625 50  0000 C CNN
-F 2 "" H 2950 3100 50  0001 C CNN
+F 2 "Pin_Headers:Pin_Header_Straight_1x03_Pitch2.54mm" H 2950 3100 50  0001 C CNN
 F 3 "" H 2950 3100 50  0001 C CNN
 	1    2950 2900
@@
 $EndComp
 $Comp
-L +3.3V #PWR2
+L +3.3V #PWR09
 U 1 1 592A5ADB
 P 3400 2500
-F 0 "#PWR2" H 3400 2350 50  0001 C CNN
+F 0 "#PWR09" H 3400 2350 50  0001 C CNN
 F 1 "+3.3V" H 3400 2640 50  0000 C CNN
 F 2 "" H 3400 2500 50  0001 C CNN
@@
 $EndComp
 $Comp
-L GND #PWR3
+L GND #PWR010
 U 1 1 592A5B0A
 P 3400 3300
-F 0 "#PWR3" H 3400 3050 50  0001 C CNN
+F 0 "#PWR010" H 3400 3050 50  0001 C CNN
 F 1 "GND" H 3400 3150 50  0000 C CNN
 F 2 "" H 3400 3300 50  0001 C CNN
@@
 	5550 4750 5550 4950
 Wire Wire Line
-	5500 1250 5500 1800
-Wire Wire Line
-	5500 1800 5500 2200
+	5500 1250 5500 2200
 $Comp
 L CONN_01X07 J4
@@
 F 0 "J4" H 8000 4050 50  0000 C CNN
 F 1 "CONN_01X07" V 8100 3650 50  0000 C CNN
-F 2 "" H 8000 3650 50  0001 C CNN
+F 2 "Pin_Headers:Pin_Header_Straight_1x07_Pitch2.54mm" H 8000 3650 50  0001 C CNN
 F 3 "" H 8000 3650 50  0001 C CNN
 	1    8000 3650
@@
 $EndComp
 $Comp
-L +3.3V #PWR12
+L +3.3V #PWR011
 U 1 1 592A6DD6
 P 7250 3200
-F 0 "#PWR12" H 7250 3050 50  0001 C CNN
+F 0 "#PWR011" H 7250 3050 50  0001 C CNN
 F 1 "+3.3V" H 7250 3340 50  0000 C CNN
 F 2 "" H 7250 3200 50  0001 C CNN
@@
 	7300 3900 6250 3900
 $Comp
-L GND #PWR11
+L GND #PWR012
 U 1 1 592A6F95
 P 7150 3600
-F 0 "#PWR11" H 7150 3350 50  0001 C CNN
+F 0 "#PWR012" H 7150 3350 50  0001 C CNN
 F 1 "GND" H 7150 3450 50  0000 C CNN
 F 2 "" H 7150 3600 50  0001 C CNN
@@
 F 0 "J2" H 6650 3750 50  0000 C CNN
 F 1 "CONN_01X06" V 6750 3400 50  0000 C CNN
-F 2 "" H 6650 3400 50  0001 C CNN
+F 2 "Pin_Headers:Pin_Header_Straight_1x06_Pitch2.54mm" H 6650 3400 50  0001 C CNN
 F 3 "" H 6650 3400 50  0001 C CNN
 	1    6650 3400
@@
 F 0 "R4" V 5230 1800 50  0000 C CNN
 F 1 "1K" V 5150 1800 50  0000 C CNN
-F 2 "" V 5080 1800 50  0001 C CNN
+F 2 "Resistors_SMD:R_0805_HandSoldering" V 5080 1800 50  0001 C CNN
 F 3 "" H 5150 1800 50  0001 C CNN
 	1    5150 1800
@@
 F 0 "D1" H 4800 2150 50  0000 C CNN
 F 1 "LED" H 4800 1950 50  0000 C CNN
-F 2 "" H 4800 2050 50  0001 C CNN
+F 2 "LEDs:LED_0805" H 4800 2050 50  0001 C CNN
 F 3 "" H 4800 2050 50  0001 C CNN
 	1    4800 2050
@@
 $EndComp
 $Comp
-L GND #PWR6
+L GND #PWR013
 U 1 1 594DDFC0
 P 4800 2300
-F 0 "#PWR6" H 4800 2050 50  0001 C CNN
+F 0 "#PWR013" H 4800 2050 50  0001 C CNN
 F 1 "GND" H 4800 2150 50  0000 C CNN
 F 2 "" H 4800 2300 50  0001 C CNN
@@
 F 0 "J3" H 6750 2800 50  0000 C CNN
 F 1 "CONN_01X02" V 6850 2650 50  0000 C CNN
-F 2 "" H 6750 2650 50  0001 C CNN
+F 2 "Pin_Headers:Pin_Header_Straight_1x02_Pitch2.54mm" H 6750 2650 50  0001 C CNN
 F 3 "" H 6750 2650 50  0001 C CNN
 	1    6750 2650
@@
 	2750 4500 2750 4650
 Wire Wire Line
-	2750 4650 3050 4650
-Wire Wire Line
-	3050 4650 3400 4650
-Wire Wire Line
-	3400 4650 3800 4650
+	2750 4650 3800 4650
 Wire Wire Line
 	3400 4850 3400 4650
@@
 F 0 "R5" V 5680 1850 50  0000 C CNN
 F 1 "0" V 5600 1850 50  0000 C CNN
-F 2 "" V 5530 1850 50  0001 C CNN
+F 2 "Resistors_SMD:R_0805_HandSoldering" V 5530 1850 50  0001 C CNN
 F 3 "" H 5600 1850 50  0001 C CNN
 	1    5600 1850
@@
 F 0 "R1" V 2830 3800 50  0000 C CNN
 F 1 "1K" V 2750 3800 50  0000 C CNN
-F 2 "" V 2680 3800 50  0001 C CNN
+F 2 "Resistors_SMD:R_0805_HandSoldering" V 2680 3800 50  0001 C CNN
 F 3 "" H 2750 3800 50  0001 C CNN
 	1    2750 3800
@@
 $EndComp
 $Comp
-L +3.3V #PWR1
+L +3.3V #PWR014
 U 1 1 594E214F
 P 2750 3600
-F 0 "#PWR1" H 2750 3450 50  0001 C CNN
+F 0 "#PWR014" H 2750 3450 50  0001 C CNN
 F 1 "+3.3V" H 2750 3740 50  0000 C CNN
 F 2 "" H 2750 3600 50  0001 C CNN
@@
 F 0 "R6" V 8830 1250 50  0000 C CNN
 F 1 "1K" V 8750 1250 50  0000 C CNN
-F 2 "" V 8680 1250 50  0001 C CNN
+F 2 "Resistors_SMD:R_0805_HandSoldering" V 8680 1250 50  0001 C CNN
 F 3 "" H 8750 1250 50  0001 C CNN
 	1    8750 1250
@@
 F 0 "D2" H 8750 1750 50  0000 C CNN
 F 1 "LED" H 8750 1550 50  0000 C CNN
-F 2 "" H 8750 1650 50  0001 C CNN
+F 2 "LEDs:LED_0805" H 8750 1650 50  0001 C CNN
 F 3 "" H 8750 1650 50  0001 C CNN
 	1    8750 1650
@@
 $EndComp
 $Comp
-L GND #PWR13
+L GND #PWR015
 U 1 1 594E29ED
 P 8750 1950
-F 0 "#PWR13" H 8750 1700 50  0001 C CNN
+F 0 "#PWR015" H 8750 1700 50  0001 C CNN
 F 1 "GND" H 8750 1800 50  0000 C CNN
 F 2 "" H 8750 1950 50  0001 C CNN

Commit message: Add meta details for crystal
Parts:
- SW1: footprint (none) -> Switches:PTS525_SM15_SMTR2_LFS
- U1: footprint (none) -> Housings_SSOP:TSSOP-20_4.4x6.5mm_Pitch0.65mm
- Y1: DKPN (none) -> 535-10212-1-ND; MPN (none) -> ABLS-8.000MHZ-B4-T
Changed lines of the file:
@@
 F 0 "U1" H 6000 2400 60  0000 C CNN
 F 1 "STM32F030x4" H 5500 3850 60  0000 C CNN
-F 2 "" H 5550 3700 60  0001 C CNN
+F 2 "Housings_SSOP:TSSOP-20_4.4x6.5mm_Pitch0.65mm" H 5550 3700 60  0001 C CNN
 F 3 "http://www.st.com/content/ccc/resource/technical/document/datasheet/a4/5d/0b/0e/87/c4/4d/71/DM00088500.pdf/files/DM00088500.pdf/jcr:content/translations/en.DM00088500.pdf" H 5550 3700 60  0001 C CNN
 F 4 "STM32F030F4P6" H 5550 3500 60  0001 C CNN "MPN"
@@
 F 1 "8MHz" H 4200 3350 50  0000 C CNN
 F 2 "" H 4200 3500 50  0001 C CNN
-F 3 "" H 4200 3500 50  0001 C CNN
+F 3 "http://www.abracon.com/Resonators/abls.pdf" H 4200 3500 50  0001 C CNN
+F 4 "ABLS-8.000MHZ-B4-T" H 4200 3500 60  0001 C CNN "MPN"
+F 5 "535-10212-1-ND" H 4200 3500 60  0001 C CNN "DKPN"
 	1    4200 3500
 	0    -1   -1   0
@@
 F 0 "SW1" H 3400 4400 60  0000 C CNN
 F 1 "PTS525-SM15" H 3400 4000 60  0000 C CNN
-F 2 "" H 3400 4200 60  0001 C CNN
+F 2 "Switches:PTS525_SM15_SMTR2_LFS" H 3400 4200 60  0001 C CNN
 F 3 "http://www.ckswitches.com/media/1467/pts525.pdf" H 3400 4200 60  0001 C CNN
 F 4 "PTS525SM15SMTR2 LFS" H 3400 4200 60  0001 C CNN "MPN"
@@
 	3750 4350 3800 4350
 Wire Wire Line
-	3800 4650 3800 4350
+	3800 4350 3800 4650
 $Comp
 L CONN_01X03_MALE J1

Commit message: Associate crystal
Parts:
- Y1: footprint (none) -> IFM-Resonators:ABLS-8.000MHZ-B4-T
Changed lines of the file:
@@
 F 0 "Y1" H 4200 3650 50  0000 C CNN
 F 1 "8MHz" H 4200 3350 50  0000 C CNN
-F 2 "" H 4200 3500 50  0001 C CNN
+F 2 "IFM-Resonators:ABLS-8.000MHZ-B4-T" H 4200 3500 50  0001 C CNN
 F 3 "http://www.abracon.com/Resonators/abls.pdf" H 4200 3500 50  0001 C CNN
 F 4 "ABLS-8.000MHZ-B4-T" H 4200 3500 60  0001 C CNN "MPN"
